Commit message: update

File: src/lab2/urdf/three_revolute.urdf (robot description, URDF)
Before this commit: robot three_revolute, 5 links, 4 joints
Joints:
- joint joint2: origin xyz=0 0 0.5 rpy=0 0 0 -> xyz=0.5 0 0 rpy=1.5708 1.5708 0
- joint joint3: origin xyz=0 0 0.5 rpy=0 0 0 -> xyz=0.2 0 0 rpy=-1.5708 0 0
